Commit message: update: UGV model is added.

File: robot_descriptions/UGV/urdf/nifti.urdf (robot description, URDF)
Before this commit: robot NIFTi, 31 links, 30 joints
Links:
- link antenna: geometry collision cylinder length=0.03718 radius=0.008; collision cylinder length=0.38107 radius=0.008
- link base_link: geometry collision box size=0.055 0.020 0.075; collision box size=0.055 0.020 0.075
- link battery: geometry collision box size=0.1450 0.1350 0.0820; visual mesh filename=../meshes/battery.dae scale=1.0 1.0 1.0
- link front_left_flipper: geometry collision box size=0.20 0.04981 0.07; collision box size=0.330000 0.04981 0.0825
- link front_right_flipper: geometry collision box size=0.20 0.04981 0.07; collision box size=0.330000 0.04981 0.0825
- link left_track: geometry collision box size=0.097000 0.178 0.500000; collision cylinder length=0.097000 radius=0.089000
- link omnicam: geometry collision cylinder length=0.137 radius=0.068; visual mesh filename=../meshes/omnicam.dae scale=1.0 1.0 1.0
- link os_sensor: geometry collision cylinder length=0.0735 radius=0.0435; visual mesh filename=../meshes/ouster-os0.dae
- link ouster_holder: geometry visual mesh filename=../meshes/ouster_holder_ladybug.dae
- link rear_left_flipper: geometry collision box size=0.20 0.04981 0.07; collision box size=0.330000 0.04981 0.055
- link rear_right_flipper: geometry collision box size=0.20 0.04981 0.07; collision box size=0.330000 0.04981 0.055
- link right_track: geometry collision box size=0.097000 0.178 0.500000; collision cylinder length=0.097000 radius=0.089000
- link top_box: geometry collision box size=0.03732 0.03523 0.03489; collision box size=0.0440 0.0440 0.01303
